Commit message: Initial commit

File: src/lekiwi/config/lekiwi.ros2_control.xacro (robot description, xacro)
@@ -1,83 +1,71 @@
 <?xml version="1.0"?>
 <robot xmlns:xacro="http://www.ros.org/wiki/xacro">
-  <xacro:macro name="lekiwi_ros2_control" params="name initial_positions_file use_fake_hardware">
+  <xacro:macro name="lekiwi_ros2_control" params="name initial_positions_file">
     <xacro:property name="initial_positions"
       value="${xacro.load_yaml(initial_positions_file)['initial_positions']}" />
     <ros2_control name="${name}" type="system">
-      <hardware>
-        <xacro:if value="${use_fake_hardware}">
-          <plugin>mock_components/GenericSystem</plugin>
-        </xacro:if>
-        <xacro:unless value="${use_fake_hardware}">
-          <plugin>lekiwi_controller/LeKiwiInterface</plugin>
-          <param name="use_serial">true</param>
-          <param name="serial_port">/dev/ttyACM0</param>
-          <param name="serial_baudrate">1000000</param>
-          <param name="joint_offsets_file">$(find lekiwi_hardware)/config/joint_offsets.yaml</param>
-        </xacro:unless>
-      </hardware>
+        <hardware>
+        <plugin>gz_ros2_control/GazeboSimSystem</plugin>
+        </hardware>
       <joint name="Shoulder_Rotation">
-        <command_interface name="position" />
-        <state_interface name="position">
-          <param name="initial_value">${initial_positions['Shoulder_Rotation']}</param>
+        <hardware_interface name="position"/> <state_interface name="position">    <param name="initial_value">${initial_positions['Shoulder_Rotation']}</param>
         </state_interface>
-        <!-- <state_interface name="velocity"/> -->
+        <state_interface name="velocity"/>
       </joint>
       <joint name="Shoulder_Pitch">
-        <command_interface name="position" />
+        <hardware_interface name="position"/>
         <state_interface name="position">
           <param name="initial_value">${initial_positions['Shoulder_Pitch']}</param>
         </state_interface>
-        <!-- <state_interface name="velocity"/> -->
+        <state_interface name="velocity"/>
       </joint>
       <joint name="Elbow">
-        <command_interface name="position" />
+        <hardware_interface name="position"/>
         <state_interface name="position">
           <param name="initial_value">${initial_positions['Elbow']}</param>
         </state_interface>
-        <!-- <state_interface name="velocity"/> -->
+        <state_interface name="velocity"/>
       </joint>
       <joint name="Wrist_Pitch">
-        <command_interface name="position" />
+        <hardware_interface name="position"/>
         <state_interface name="position">
           <param name="initial_value">${initial_positions['Wrist_Pitch']}</param>
         </state_interface>
-        <!-- <state_interface name="velocity"/> -->
+        <state_interface name="velocity"/>
       </joint>
       <joint name="Wrist_Roll">
-        <command_interface name="position" />
+        <hardware_interface name="position"/>
         <state_interface name="position">
           <param name="initial_value">${initial_positions['Wrist_Roll']}</param>
         </state_interface>
-        <!-- <state_interface name="velocity"/> -->
+        <state_interface name="velocity"/>
       </joint>
       <joint name="Gripper">
-        <command_interface name="position" />
+        <hardware_interface name="position"/>
         <state_interface name="position">
           <param name="initial_value">${initial_positions['Gripper']}</param>
         </state_interface>
-        <!-- <state_interface name="velocity"/> -->
+        <state_interface name="velocity"/>
       </joint>
-      <!-- WHEEL JOINTS (Motor IDs 7-9) - Use velocity control -->
       <joint name="left_wheel_drive">
-        <command_interface name="velocity" />
+        <hardware_interface name="velocity"/>
         <state_interface name="position">
-          <param name="initial_value">${initial_positions['left_wheel_drive']}</param>
+          <param name="initial_value">0.0</param>
         </state_interface>
-        <state_interface name="velocity" />
+        <state_interface name="velocity"/>
       </joint>
       <joint name="rear_wheel_drive">
-        <command_interface name="velocity" />
+        <hardware_interface name="velocity"/>
         <state_interface name="position">
-          <param name="initial_value">${initial_positions['rear_wheel_drive']}</param>
+          <param name="initial_value">0.0</param>
         </state_interface>
-        <state_interface name="velocity" />
+        <state_interface name="velocity"/>
       </joint>
       <joint name="right_wheel_drive">
-        <command_interface name="velocity" />
+        <hardware_interface name="velocity"/>
         <state_interface name="position">
-          <param name="initial_value">${initial_positions['right_wheel_drive']}</param>
+          <param name="initial_value">0.0</param>
         </state_interface>
-        <state_interface name="velocity" />
+        <state_interface name="velocity"/>
       </joint>
     </ros2_control>

File: src/lekiwi/config/lekiwi.urdf.xacro (robot description, xacro)
@@ -2,21 +2,15 @@
 <robot xmlns:xacro="http://www.ros.org/wiki/xacro" name="lekiwi">
     <xacro:arg name="initial_positions_file" default="initial_positions.yaml" />
-    <xacro:arg name="use_fake_hardware" default="false" />
-    <!-- Import lekiwi mobile base urdf file (includes proper base frame connections) -->
     <xacro:include filename="$(find lekiwi)/urdf/lekiwi_complete.urdf" />
-    <!-- Import control_xacro -->
-    <xacro:include filename="lekiwi.ros2_control.xacro" />
-    <!-- Add base_footprint as the root frame with proper orientation -->
-    <!-- This aligns the coordinate system: X=forward, Y=left, Z=up -->
     <link name="base_footprint" />
     <joint name="base_footprint_joint" type="fixed">
         <parent link="base_footprint" />
         <child link="base_link" />
-        <!-- Apply 90-degree rotation to align coordinate frames: X=forward, Y=left -->
-        <origin xyz="0 0 0" rpy="0 0 -1.5708" />
+        <origin xyz="0.0 0.0 0.026" rpy="0 0 0" />
     </joint>
+    <xacro:include filename="$(find lekiwi)/config/lekiwi.ros2_control.xacro" />
     <xacro:lekiwi_ros2_control
         name="SO100ARM"
         initial_positions_file="$(arg initial_positions_file)"
-        use_fake_hardware="$(arg use_fake_hardware)" />
-</robot>
+        />
+    </robot>

File: src/lekiwi/urdf/lekiwi.urdf (robot description, URDF)
Before this commit: robot lekiwi, 8 links, 7 joints
Links:
- link Base: geometry collision mesh filename=model://lekiwi/models/lekiwi_5dof/meshes/Base.STL; visual mesh filename=model://lekiwi/models/lekiwi_5dof/meshes/Base.STL
- link Fixed_Gripper: geometry collision mesh filename=model://lekiwi/models/lekiwi_5dof/meshes/Fixed_Gripper.STL; visual mesh filename=model://lekiwi/models/lekiwi_5dof/meshes/Fixed_Gripper.STL
- link Lower_Arm: geometry collision mesh filename=model://lekiwi/models/lekiwi_5dof/meshes/Lower_Arm.STL; visual mesh filename=model://lekiwi/models/lekiwi_5dof/meshes/Lower_Arm.STL
- link Moving_Jaw: geometry collision mesh filename=model://lekiwi/models/lekiwi_5dof/meshes/Moving_Jaw.STL; visual mesh filename=model://lekiwi/models/lekiwi_5dof/meshes/Moving_Jaw.STL
- link Shoulder_Rotation_Pitch: geometry collision mesh filename=model://lekiwi/models/lekiwi_5dof/meshes/Shoulder_Rotation_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; visual mesh filename=model://lekiwi/models/lekiwi_5dof/meshes/Shoulder_Rotation_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
- link Upper_Arm: geometry collision mesh filename=model://lekiwi/models/lekiwi_5dof/meshes/Upper_Arm.STL; visual mesh filename=model://lekiwi/models/lekiwi_5dof/meshes/Upper_Arm.STL
- link Wrist_Pitch_Roll: geometry collision mesh filename=model://lekiwi/models/lekiwi_5dof/meshes/Wrist_Pitch_Roll.S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; visual mesh filename=model://lekiwi/models/lekiwi_5dof/meshes/Wrist_Pitch_Roll.S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

File: src/lekiwi/urdf/lekiwi_5dof.urdf (robot description, URDF)
Before this commit: robot lekiwi, 8 links, 7 joints
Links:
- link Base_08q-v1: geometry collision mesh filename=model://lekiwi/models/lekiwi_5dof/meshes/Base.STL; visual mesh filename=model://lekiwi/models/lekiwi_5dof/meshes/Base.STL
- link Fixed_Gripper: geometry collision mesh filename=model://lekiwi/models/lekiwi_5dof/meshes/Fixed_Gripper.STL scale=0.9 0.9 0.9; visual mesh filename=model://lekiwi/models/lekiwi_5dof/meshes/Fixed_Gripper.STL
- link Lower_Arm: geometry collision mesh filename=model://lekiwi/models/lekiwi_5dof/meshes/Lower_Arm.STL scale=0.9 0.9 0.9; visual mesh filename=model://lekiwi/models/lekiwi_5dof/meshes/Lower_Arm.STL
- link Moving_Jaw: geometry collision mesh filename=model://lekiwi/models/lekiwi_5dof/meshes/Moving_Jaw.STL scale=0.9 0.9 0.9; visual mesh filename=model://lekiwi/models/lekiwi_5dof/meshes/Moving_Jaw.STL
- link Shoulder_Rotation_Pitch: geometry collision mesh filename=model://lekiwi/models/lekiwi_5dof/meshes/Shoulder_Rotation_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 scale=0.9 0.9 0.9; visual mesh filename=model://lekiwi/models/lekiwi_5dof/meshes/Shoulder_Rotation_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
- link Upper_Arm: geometry collision mesh filename=model://lekiwi/models/lekiwi_5dof/meshes/Upper_Arm.STL scale=0.9 0.9 0.9; visual mesh filename=model://lekiwi/models/lekiwi_5dof/meshes/Upper_Arm.STL
- link Wrist_Pitch_Roll: geometry collision mesh filename=model://lekiwi/models/lekiwi_5dof/meshes/Wrist_Pitch_Roll.S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 scale=0.9 0.9 0.9; visual mesh filename=model://lekiwi/models/lekiwi_5dof/meshes/Wrist_Pitch_Roll.S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

File: src/lekiwi/urdf/so_100_arm_5dof.urdf (robot description, URDF)
Before this commit: robot lekiwi, 8 links, 7 joints
Links:
- link Base: geometry collision mesh filename=model://lekiwi/models/lekiwi_5dof/meshes/Base.STL; visual mesh filename=model://lekiwi/models/lekiwi_5dof/meshes/Base.STL
- link Fixed_Gripper: geometry collision mesh filename=model://lekiwi/models/lekiwi_5dof/meshes/Fixed_Gripper.STL; visual mesh filename=model://lekiwi/models/lekiwi_5dof/meshes/Fixed_Gripper.STL
- link Lower_Arm: geometry collision mesh filename=model://lekiwi/models/lekiwi_5dof/meshes/Lower_Arm.STL; visual mesh filename=model://lekiwi/models/lekiwi_5dof/meshes/Lower_Arm.STL
- link Moving_Jaw: geometry collision mesh filename=model://lekiwi/models/lekiwi_5dof/meshes/Moving_Jaw.STL; visual mesh filename=model://lekiwi/models/lekiwi_5dof/meshes/Moving_Jaw.STL
- link Shoulder_Rotation_Pitch: geometry collision mesh filename=model://lekiwi/models/lekiwi_5dof/meshes/Shoulder_Rotation_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; visual mesh filename=model://lekiwi/models/lekiwi_5dof/meshes/Shoulder_Rotation_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
- link Upper_Arm: geometry collision mesh filename=model://lekiwi/models/lekiwi_5dof/meshes/Upper_Arm.STL; visual mesh filename=model://lekiwi/models/lekiwi_5dof/meshes/Upper_Arm.STL
- link Wrist_Pitch_Roll: geometry collision mesh filename=model://lekiwi/models/lekiwi_5dof/meshes/Wrist_Pitch_Roll.S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; visual mesh filename=model://lekiwi/models/lekiwi_5dof/meshes/Wrist_Pitch_Roll.S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
